Commit message: golden commit 2

File: putarm_ur3e/urdf/putarm_ur3e.xacro (robot description, xacro)
@@ -80,6 +80,6 @@
   </joint>
   <xacro:sensor_d435 parent="d435_link" name="intel_cam" >
-    <origin xyz="0.0 0.065 0.013" rpy="1.570 -1.570 3.140"/>
-     <!-- <origin xyz="0.0 0.08 0.0155" rpy="0 0 0"/> -->
+    <!--<origin xyz="0.0 0.065 0.013" rpy="1.570 -1.570 3.140"/>-->
+     <origin xyz="0.0 0.0905 0.013" rpy="1.570 -1.570 0"/>
   </xacro:sensor_d435>
   <link name="dumb_link">

Commit message: 67 kwietnia

File: putarm_ur3e/urdf/putarm_ur3e.xacro (robot description, xacro)
@@ -99,4 +99,12 @@
     <child link="dumb_link_2"/>
   </joint>
+  <link name="dumb_link_3">
+    <origin xyz="0.0 0.0 0.0" rpy="0 0 0"/>
+  </link>
+  <joint name="dumb_joint_3" type="fixed">
+    <origin xyz="0.032 -0.0779 0.0" rpy="0.0 0 0" />
+    <parent link="dumb_link_2"/>
+    <child link="dumb_link_3"/>
+  </joint>
   <link name="gripper">
     <visual>
